Commit message: minor changes xacro: parent name with added '_link' in ouster (for add on other robots) plugin: add info

File: ouster_os1_64/urdf/example_robot.urdf.xacro (robot description, xacro)
@@ -2,5 +2,5 @@
 <robot xmlns:xacro="http://ros.org/wiki/xacro" name="example_robot">
   <!-- Base Footprint -->
-  <link name="base_footprint" />
+  <link name="base_footprint_link" />
   <xacro:include filename="$(find ouster_os1_64)/urdf/os1_64.urdf.xacro"/>
   <os1_64 parent="base_footprint" name="ouster" prefix="/os1_cloud_node" hz="10" samples="512">

File: ouster_os1_64/urdf/os1_64.urdf.xacro (robot description, xacro)
@@ -3,8 +3,8 @@
 <robot xmlns:xacro="http://ros.org/wiki/xacro" name="os1_64">
   <xacro:property name="PI" value="3.1415926535897931"/>
-  <xacro:macro name="os1_64" params="*origin parent:=base_link name:=ouster prefix:=/os1_cloud_node hz:=10 samples:=512 min_range:=0.8 max_range:=100 noise:=0.008 min_angle_v:=-16.6 max_angle_v:=16.6">
-    <joint name="${name}_base_mount_joint" type="fixed">
+  <xacro:macro name="os1_64" params="*origin parent:=base name:=ouster prefix:=/os1_cloud_node hz:=10 samples:=512 min_range:=0.8 max_range:=100 noise:=0.008 min_angle_v:=-16.6 max_angle_v:=16.6">
+    <joint name="${name}_joint" type="fixed">
       <xacro:insert_block name="origin" />
-      <parent link="${parent}"/>
+      <parent link="${parent}_link"/>
       <child link="${name}_sensor"/>
     </joint>
