Commit message: [ouster_os1_64] frame architecture and dae file

File: ouster_os1_64/urdf/os1_64.urdf.xacro (robot description, xacro)
@@ -7,7 +7,7 @@
       <xacro:insert_block name="origin" />
       <parent link="${parent}"/>
-      <child link="${name}"/>
+      <child link="${name}_sensor"/>
     </joint>
-    <link name="${name}">
+    <link name="${name}_sensor">
       <inertial>
         <mass value="0.425"/>
@@ -25,11 +25,18 @@
         <origin xyz="0 0 0" rpy="0 0 0"/>
         <geometry>
-          <mesh filename="package://ouster_os1_64/meshes/os1_64.stl"/>
+          <mesh filename="package://ouster_os1_64/meshes/os1_64.dae" scale="0.001 0.001 0.001" />
         </geometry>
       </visual>
     </link>
-    <gazebo reference="${name}">
+    <link name="${name}_lidar">
+      <pose>0 0 0 0 0 ${PI}</pose>
+    </link>
+    <joint name="${name}_lidar_joint" type="fixed">
+      <parent link="${name}_sensor"/>
+      <child link="${name}_lidar"/>
+    </joint>
+    <gazebo reference="${name}_lidar">
       <sensor type="ray" name="${name}_lidar">
-        <pose>0 0 0 0 0 ${PI}</pose>
+        <pose>0 0 0 0 0 0</pose>
         <visualize>false</visualize>
         <update_rate>${hz}</update_rate>
@@ -62,5 +69,5 @@
         <plugin name="gazebo_ros_laser_controller" filename="libgazebo_ros_ouster_laser.so">
           <topicName>${prefix}/points</topicName>
-          <frameName>${name}</frameName>
+          <frameName>${name}_lidar</frameName>
           <min_range>${min_range}</min_range>
           <max_range>${max_range}</max_range>
@@ -71,5 +78,5 @@
     <link name="${name}_imu"/>
     <joint name="${name}_imu_joint" type="fixed">
-      <parent link="${name}"/>
+      <parent link="${name}_sensor"/>
       <child link="${name}_imu"/>
     </joint>

Commit message: Model: update mesh modify scale of main meshes and add reduced meshes

File: ouster_os1_64/urdf/os1_64.urdf.xacro (robot description, xacro)
@@ -3,5 +3,12 @@
 <robot xmlns:xacro="http://ros.org/wiki/xacro" name="os1_64">
   <xacro:property name="PI" value="3.1415926535897931"/>
-  <xacro:macro name="os1_64" params="*origin parent:=base name:=ouster prefix:=/os1_cloud_node hz:=10 samples:=512 min_range:=0.8 max_range:=100 noise:=0.008 min_angle_v:=-16.6 max_angle_v:=16.6">
+  <xacro:macro name="os1_64" params="*origin parent:=base name:=ouster reduced:=true prefix:=/os1_cloud_node hz:=10 samples:=512 min_range:=0.8 max_range:=100 noise:=0.008 min_angle_v:=-16.6 max_angle_v:=16.6">
+    <!-- Conditional properties -->
+    <xacro:if value="${reduced}">
+      <xacro:property name="file_visual" value="os1_64_reduced"/>
+    </xacro:if>
+    <xacro:unless value="${reduced}">
+      <xacro:property name="file_visual" value="os1_64"/>
+    </xacro:unless>
     <joint name="${name}_joint" type="fixed">
       <xacro:insert_block name="origin" />
@@ -16,5 +23,5 @@
                  iyy="0.000308429" iyz="0" izz="0.00034589"/>
       </inertial>
-      <collision name="base_collision">
+      <collision name="lidar_collision">
         <origin xyz="0 0 0.03675" rpy="0 0 0" />
         <geometry>
@@ -22,8 +29,8 @@
         </geometry>
       </collision>
-      <visual name="base_visual">
+      <visual name="lidar_visual">
         <origin xyz="0 0 0" rpy="0 0 0"/>
         <geometry>
-          <mesh filename="package://ouster_os1_64/meshes/os1_64.dae" scale="0.001 0.001 0.001" />
+          <mesh filename="package://ouster_os1_64/meshes/${file_visual}.stl" />
         </geometry>
       </visual>

Commit message: Fix gpu usage GPU can now be used for lidar simulation

File: ouster_os1_64/urdf/os1_64.urdf.xacro (robot description, xacro)
@@ -3,5 +3,5 @@
 <robot xmlns:xacro="http://ros.org/wiki/xacro" name="os1_64">
   <xacro:property name="PI" value="3.1415926535897931"/>
-  <xacro:macro name="os1_64" params="*origin parent:=base name:=ouster reduced:=true prefix:=/os1_cloud_node hz:=10 samples:=512 min_range:=0.8 max_range:=100 noise:=0.008 min_angle_v:=-16.6 max_angle_v:=16.6">
+  <xacro:macro name="os1_64" params="*origin parent:=base name:=ouster reduced:=true prefix:=/os1_cloud_node hz:=10 samples:=512 min_range:=0.8 max_range:=100 noise:=0.008 min_angle_v:=-16.6 max_angle_v:=16.6 gpu:=false">
     <!-- Conditional properties -->
     <xacro:if value="${reduced}">
@@ -10,4 +10,10 @@
     <xacro:unless value="${reduced}">
       <xacro:property name="file_visual" value="os1_64"/>
+    </xacro:unless>
+    <xacro:if value="${gpu}">
+      <xacro:property name="gpu_str" value="gpu_"/>
+    </xacro:if>
+    <xacro:unless value="${gpu}">
+      <xacro:property name="gpu_str" value=""/>
     </xacro:unless>
     <joint name="${name}_joint" type="fixed">
@@ -44,5 +50,5 @@
     </joint>
     <gazebo reference="${name}_lidar">
-      <sensor type="ray" name="${name}_lidar">
+      <sensor type="${gpu_str}ray" name="${name}_lidar">
         <pose>0 0 0 0 0 0</pose>
         <visualize>false</visualize>
@@ -74,5 +80,5 @@
           </noise>
         </ray>
-        <plugin name="gazebo_ros_laser_controller" filename="libgazebo_ros_ouster_laser.so">
+        <plugin name="gazebo_ros_laser_controller" filename="libgazebo_ros_ouster_${gpu_str}laser.so">
           <topicName>${prefix}/points</topicName>
           <frameName>${name}_lidar</frameName>
